File: kicad/esp32-s3-utility-carrier.kicad_sch (KiCad schematic)
At the start: 27 parts, among them SW1 BTN1, SW2 BTN2, SW3 BTN3, U2 SN74AHCT125N

Commit message: fix(pcb): reset placeholder layout for readability
v0.4: 110x75 mm board, grouped placement, minimal keep-outs,
no copper pours or tracks, small zone silk labels only.

Co-authored-by: Cursor <cursoragent@cursor.com>
Other:
- note added: "PLACEHOLDER SCHEMATIC v0.4 - run ERC in KiCad ESP32 footprint NOT FINAL - see measurements.md Do NOT order PCB / no Gerbers"
- note removed: "PLACEHOLDER SCHEMATIC v0.3 - run ERC in KiCad ESP32 footprint NOT FINAL - see measurements.md Do NOT order PCB / no Gerbers"
Changed lines of the file:
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@@
     (title "ESP32-S3 Utility Carrier v1")
     (date "2026-05-21")
-    (rev "0.3-placeholder")
+    (rev "0.4-placeholder")
     (comment 1 "NOT FOR PRODUCTION - ESP footprint NOT FINAL")
     (comment 2 "See hardware/measurements.md before ordering PCB")
@@
   )  (text "W5500 OPTIONAL / NOT POPULATED\nBedrade module voor toekomstige Art-Net/sACN route\nSPI: GPIO5/13/14 CS47 RST4 INT39 (zie pinout-table.md)"
     (at 295 43 0) (effects (font (size 1.2 1.2)) (justify left)))
-  (text "PLACEHOLDER SCHEMATIC v0.3 - run ERC in KiCad\nESP32 footprint NOT FINAL - see measurements.md\nDo NOT order PCB / no Gerbers"
+  (text "PLACEHOLDER SCHEMATIC v0.4 - run ERC in KiCad\nESP32 footprint NOT FINAL - see measurements.md\nDo NOT order PCB / no Gerbers"
     (at 30 30 0) (effects (font (size 1.5 1.5)) (justify left)))
   (sheet_instances
-    (path "/a3d7de30-62c7-4e8d-8a95-f8503270e9ba" (page "1"))
+    (path "/b7c9fba0-129e-478c-8ad9-638c6e8e49a3" (page "1"))
   )
 )

Commit message: feat(pcb): align layout to zone diagram
v0.5: 130x85 mm board, six dashed zone guides, component placement
per user diagram; airwires only, no copper pours.

Co-authored-by: Cursor <cursoragent@cursor.com>
Other:
- note added: "PLACEHOLDER SCHEMATIC v0.5 - run ERC in KiCad ESP32 footprint NOT FINAL - see measurements.md Do NOT order PCB / no Gerbers"
- note removed: "PLACEHOLDER SCHEMATIC v0.4 - run ERC in KiCad ESP32 footprint NOT FINAL - see measurements.md Do NOT order PCB / no Gerbers"
Changed lines of the file:
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@@
     (title "ESP32-S3 Utility Carrier v1")
     (date "2026-05-21")
-    (rev "0.4-placeholder")
+    (rev "0.5-placeholder")
     (comment 1 "NOT FOR PRODUCTION - ESP footprint NOT FINAL")
     (comment 2 "See hardware/measurements.md before ordering PCB")
@@
   )  (text "W5500 OPTIONAL / NOT POPULATED\nBedrade module voor toekomstige Art-Net/sACN route\nSPI: GPIO5/13/14 CS47 RST4 INT39 (zie pinout-table.md)"
     (at 295 43 0) (effects (font (size 1.2 1.2)) (justify left)))
-  (text "PLACEHOLDER SCHEMATIC v0.4 - run ERC in KiCad\nESP32 footprint NOT FINAL - see measurements.md\nDo NOT order PCB / no Gerbers"
+  (text "PLACEHOLDER SCHEMATIC v0.5 - run ERC in KiCad\nESP32 footprint NOT FINAL - see measurements.md\nDo NOT order PCB / no Gerbers"
     (at 30 30 0) (effects (font (size 1.5 1.5)) (justify left)))
   (sheet_instances
-    (path "/b7c9fba0-129e-478c-8ad9-638c6e8e49a3" (page "1"))
+    (path "/c34b4b73-7a1f-4cba-ae2b-92890bd69a09" (page "1"))
   )
 )

Commit message: fix(pcb): place components by explicit coordinates
v0.6: PCB_PLACE/PCB_SILK drive 130×85 mm layout with overlap checks;
F_ESP x=45 for J_I2C clearance; silk nudges documented in layout plan.

Co-authored-by: Cursor <cursoragent@cursor.com>
Other:
- note added: "PLACEHOLDER SCHEMATIC v0.6 - run ERC in KiCad ESP32 footprint NOT FINAL - see measurements.md Do NOT order PCB / no Gerbers"
- note removed: "PLACEHOLDER SCHEMATIC v0.5 - run ERC in KiCad ESP32 footprint NOT FINAL - see measurements.md Do NOT order PCB / no Gerbers"
Changed lines of the file:
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@@
     (title "ESP32-S3 Utility Carrier v1")
     (date "2026-05-21")
-    (rev "0.5-placeholder")
+    (rev "0.6-placeholder")
     (comment 1 "NOT FOR PRODUCTION - ESP footprint NOT FINAL")
     (comment 2 "See hardware/measurements.md before ordering PCB")
@@
   )  (text "W5500 OPTIONAL / NOT POPULATED\nBedrade module voor toekomstige Art-Net/sACN route\nSPI: GPIO5/13/14 CS47 RST4 INT39 (zie pinout-table.md)"
     (at 295 43 0) (effects (font (size 1.2 1.2)) (justify left)))
-  (text "PLACEHOLDER SCHEMATIC v0.5 - run ERC in KiCad\nESP32 footprint NOT FINAL - see measurements.md\nDo NOT order PCB / no Gerbers"
+  (text "PLACEHOLDER SCHEMATIC v0.6 - run ERC in KiCad\nESP32 footprint NOT FINAL - see measurements.md\nDo NOT order PCB / no Gerbers"
     (at 30 30 0) (effects (font (size 1.5 1.5)) (justify left)))
   (sheet_instances
-    (path "/2d24bff7-8440-4dd0-b7ea-9da512bc4ed1" (page "1"))
+    (path "/b5628ec7-cf80-4466-9a23-c284788e228a" (page "1"))
   )
 )

Commit message: fix(pcb): align placement plan and add visible routing
v0.7: approved zone layout in PCB_PLACE, partial F.Cu routing for
LED/servo/main power, W5500 5 mm margin, overlap-checked silk.

Co-authored-by: Cursor <cursoragent@cursor.com>
Other:
- note added: "PLACEHOLDER SCHEMATIC v0.7 - run ERC in KiCad ESP32 footprint NOT FINAL - see measurements.md Do NOT order PCB / no Gerbers"
- note removed: "PLACEHOLDER SCHEMATIC v0.6 - run ERC in KiCad ESP32 footprint NOT FINAL - see measurements.md Do NOT order PCB / no Gerbers"
Changed lines of the file:
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@@
     (title "ESP32-S3 Utility Carrier v1")
     (date "2026-05-21")
-    (rev "0.6-placeholder")
+    (rev "0.7-placeholder")
     (comment 1 "NOT FOR PRODUCTION - ESP footprint NOT FINAL")
     (comment 2 "See hardware/measurements.md before ordering PCB")
@@
   )  (text "W5500 OPTIONAL / NOT POPULATED\nBedrade module voor toekomstige Art-Net/sACN route\nSPI: GPIO5/13/14 CS47 RST4 INT39 (zie pinout-table.md)"
     (at 295 43 0) (effects (font (size 1.2 1.2)) (justify left)))
-  (text "PLACEHOLDER SCHEMATIC v0.6 - run ERC in KiCad\nESP32 footprint NOT FINAL - see measurements.md\nDo NOT order PCB / no Gerbers"
+  (text "PLACEHOLDER SCHEMATIC v0.7 - run ERC in KiCad\nESP32 footprint NOT FINAL - see measurements.md\nDo NOT order PCB / no Gerbers"
     (at 30 30 0) (effects (font (size 1.5 1.5)) (justify left)))
   (sheet_instances
-    (path "/b5628ec7-cf80-4466-9a23-c284788e228a" (page "1"))
+    (path "/0469d8f2-cdbe-4dea-bd0f-2b7631f2f2a6" (page "1"))
   )
 )

Commit message: fix(pcb): replace messy routing with LED data routing only
Revert v0.7 board-wide power traces; keep v0.7 placement. Route thin
LED data chain and short C_AHCT at U2 with 45° bends outside ESP keep-outs.

Co-authored-by: Cursor <cursoragent@cursor.com>
Other:
- note added: "PLACEHOLDER SCHEMATIC v0.8 - run ERC in KiCad ESP32 footprint NOT FINAL - see measurements.md Do NOT order PCB / no Gerbers"
- note removed: "PLACEHOLDER SCHEMATIC v0.7 - run ERC in KiCad ESP32 footprint NOT FINAL - see measurements.md Do NOT order PCB / no Gerbers"
Changed lines of the file:
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@@
     (title "ESP32-S3 Utility Carrier v1")
     (date "2026-05-21")
-    (rev "0.7-placeholder")
+    (rev "0.8-placeholder")
     (comment 1 "NOT FOR PRODUCTION - ESP footprint NOT FINAL")
     (comment 2 "See hardware/measurements.md before ordering PCB")
@@
   )  (text "W5500 OPTIONAL / NOT POPULATED\nBedrade module voor toekomstige Art-Net/sACN route\nSPI: GPIO5/13/14 CS47 RST4 INT39 (zie pinout-table.md)"
     (at 295 43 0) (effects (font (size 1.2 1.2)) (justify left)))
-  (text "PLACEHOLDER SCHEMATIC v0.7 - run ERC in KiCad\nESP32 footprint NOT FINAL - see measurements.md\nDo NOT order PCB / no Gerbers"
+  (text "PLACEHOLDER SCHEMATIC v0.8 - run ERC in KiCad\nESP32 footprint NOT FINAL - see measurements.md\nDo NOT order PCB / no Gerbers"
     (at 30 30 0) (effects (font (size 1.5 1.5)) (justify left)))
   (sheet_instances
-    (path "/0469d8f2-cdbe-4dea-bd0f-2b7631f2f2a6" (page "1"))
+    (path "/0ff9db8c-a0fb-4b01-9c32-e8cbc42c4c58" (page "1"))
   )
 )

Commit message: refactor(pcb): simplify carrier around external controls and 3 LED outputs
Co-authored-by: Cursor <cursoragent@cursor.com>
Parts:
- removed F_OLED: OLED_DIRECT, Connector_PinHeader_2.54mm:PinHeader_1x04_P2.54mm_Vertical, symbol Connector:Conn_01x04_Pin
- removed J_LED4: LED4 5V|GND|DATA, carrier:JST_XH_1x03_Placeholder, symbol Connector:Conn_01x03_Pin
- removed R_LED4: 330, Resistor_THT:R_AXIAL-0.4_D5.1mm_L12.0mm_Horizontal, symbol Device:R
- removed SW1: BTN1, Button_Switch_THT:SW_PUSH_6mm, symbol Switch:SW_Push
- removed SW2: BTN2, Button_Switch_THT:SW_PUSH_6mm, symbol Switch:SW_Push
- removed SW3: BTN3, Button_Switch_THT:SW_PUSH_6mm, symbol Switch:SW_Push
- J_LED1, J_LED2, J_LED3: footprint carrier:JST_XH_1x03_Placeholder -> carrier:ScrewTerm_3p_5.08_Placeholder
- J_MAIN: footprint carrier:JST_VH_1x02_Placeholder -> carrier:ScrewTerm_2p_5.08_Placeholder
- J_W5500: footprint carrier:JST_W5500_1x08_Placeholder -> carrier:W5500_SBC_USR_ES1_Placeholder
Other:
- note added: "PLACEHOLDER SCHEMATIC v0.9 phase2 - run ERC in KiCad DevKitC-1 dims assumed — verify clone (measurements.md) Do NOT order PCB / no Gerbers"
- note added: "SBC-USR-ES1 W5500 OPTIONAL / NOT POPULATED Module 23x29mm — header TBD, measure before fab RJ45 toward board edge · SPI GPIO5/13/14/47/4/39"
- note added: "U2 ch4 (4A/4Y) DNP — NC GPIO12 free on DevKit"
- note removed: "PLACEHOLDER SCHEMATIC v0.8 - run ERC in KiCad ESP32 footprint NOT FINAL - see measurements.md Do NOT order PCB / no Gerbers"
- note removed: "W5500 OPTIONAL / NOT POPULATED Bedrade module voor toekomstige Art-Net/sACN route SPI: GPIO5/13/14 CS47 RST4 INT39 (zie pinout-table.md)"
